File: camy_cam.kicad_pcb (KiCad board)
At the start: 2 copper layers, 78.5 x 73.4 mm, 18 parts, among them J1 Conn_01x08, J2 Conn_01x02, J3 Conn_02x09_Odd_Even, SW1 SW_Push, SW2 SW_Push, SW3 SW_SPDT, U1 ESP32-S3-WROOM-1, U2 AMS1117-3.3, U3 254

Commit message: initial_commit
Parts:
- added C7: 100nF, Capacitor_THT:C_Disc_D5.0mm_W2.5mm_P5.00mm, F.Cu at (149.8, 109.2)
- added C8: 100nF, Capacitor_THT:C_Disc_D5.0mm_W2.5mm_P5.00mm, F.Cu at (149.8, 113.3)
- added R3: 10kΩ, Resistor_THT:R_Axial_DIN0207_L6.3mm_D2.5mm_P7.62mm_Horizontal, F.Cu at (139.2, 105.2)
- added R5: 4.7kΩ, Resistor_THT:R_Axial_DIN0207_L6.3mm_D2.5mm_P7.62mm_Horizontal, F.Cu at (166.3, 106.5)
- added R6: 4.7kΩ, Resistor_THT:R_Axial_DIN0207_L6.3mm_D2.5mm_P7.62mm_Horizontal, F.Cu at (166.4, 116.2)
- SW3: value SW_SPDT -> SW_Push_DPDT
- moved SW3 6.35 mm to (139.9, 108.5)
- moved C6 1.39 mm to (136.9, 117.2)
Connections:
- C4 pad 1: Net-(SW3-B) -> Net-(J2-Pin_1)
- J2 pad 1: GND -> Net-(J2-Pin_1)
- J2 pad 2: Net-(J2-Pin_2) -> GND
- SW3 pad 1: Net-(J2-Pin_2) -> GND
- SW3 pad 2: Net-(SW3-B) -> Net-(J2-Pin_1)
- SW3 pad 3: unconnected-(SW3-C-Pad3) -> GND
- SW3 pad 4: (no net) -> GND
- SW3 pad 5: (no net) -> GND
- SW3 pad 6: (no net) -> GND
- U1 pad 15: /CAM_SIOC -> Net-(U1-IO3)
- U1 pad 38: /CAM_SIOD -> Net-(U1-IO2)
- U2 pad 3: Net-(SW3-B) -> Net-(J2-Pin_1)
Routing:
- net Net-(J2-Pin_1): track 0.00 -> 95.1 mm, vias 0 -> 4
- net Net-(U1-IO3): track 0.00 -> 83.1 mm, vias 0 -> 4
- net Net-(U1-IO2): track 0.00 -> 76.6 mm, vias 0 -> 1
- net GND: track 198.3 -> 271.4 mm, vias 2 -> 10
- net /CAM_SIOC: track 9.43 -> 78.8 mm, vias 0 -> 1
- net Net-(J2-Pin_2): track 59.6 -> 0.00 mm
- net Net-(SW3-B): track 49.2 -> 0.00 mm, vias 1 -> 0
- net Net-(R3-Pad1): track 6.50 -> 53.0 mm, vias 0 -> 1
- net /CAM_SIOD: track 29.5 -> 75.2 mm
- net /3V3: track 139.9 -> 176.9 mm, vias 6 -> 10
- net /CAM_VSYNC: track 25.8 -> 44.5 mm, vias 2 -> 4
- net Net-(U1-IO0): track 0.00 -> 15.6 mm, vias 0 -> 2
- net /MISO: track 134.1 -> 129.6 mm
- net /CAM_PWDN: track 38.5 -> 39.8 mm
- net /CAM_RESET: track 26.1 -> 27.0 mm
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Other:
- board size 78.5 x 73.4 mm -> 79.9 x 73.4 mm
